File: board-kicad/VineBadge2020.kicad_pcb (KiCad board)
At the start: 2 copper layers, 95.7 x 96.4 mm, 72 parts, among them IC1 ATTINY20-X, P1 CONN_01X05, Q1 Q_NMOS_DGS

Commit message: guess I forgot to commit
Parts:
- removed G***: LOGO, LOGO
- moved D37 122.3 mm to (104.0, 108.8), turned to 90 degrees
- moved D21 115.0 mm to (115.4, 109.2), turned to 270 degrees
- moved D23 108.2 mm to (115.4, 112.2), turned to 270 degrees
- moved D2 106.6 mm to (104.0, 115.2), turned to 90 degrees
- moved D32 94.2 mm to (104.0, 121.6), turned to 90 degrees
- moved D33 94.0 mm to (122.4, 109.4), turned to 225 degrees
- moved D42 93.2 mm to (118.0, 117.0), turned to 315 degrees
- moved D46 92.6 mm to (115.4, 121.6), turned to 90 degrees
- moved D45 92.5 mm to (122.4, 121.4), turned to 135 degrees
- moved D51 91.3 mm to (120.2, 119.2), turned to 315 degrees
- moved D53 87.4 mm to (104.0, 118.4), turned to 90 degrees
- moved D29 86.0 mm to (115.4, 118.4), turned to 90 degrees
- moved D1 84.3 mm to (104.0, 112.0), turned to 90 degrees
- moved D3 82.7 mm to (115.4, 115.2), turned to 270 degrees
- moved D17 81.4 mm to (120.2, 111.6), turned to 45 degrees
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Routing:
- added copper zone on F.Cu, net GND
Other:
- outline, holes or cut-outs redrawn
