File: board-kicad/spang_badge.sch (KiCad schematic (older format))
At the start: 25 parts, among them IC1 ATTINY20-X

Commit message: ordered some parts to experiment
Parts:
- removed Q?: Q_NMOS_GSD, symbol Q_NMOS_GSD
- F1: renamed from F?; footprint (none) -> Fuse_Holders_and_Fuses:Fuse_SMD1206_HandSoldering
- IC1: footprint (none) -> spang_badge:ATTINY20_SOIC-14
- SW1: renamed from SW?; footprint (none) -> Buttons_Switches_SMD:SW_SPST_EVQPE1
- gave numbers to parts that had none: 9
Connections:
- wire segments 60 -> 58

Commit message: starting LED placement
Parts:
- BT1: footprint (none) -> spang_badge:COINCELL_20MM
Changed lines of the file:
@@
 F 0 "BT1" H 3050 5300 50  0000 L CNN
 F 1 "Battery_Cell" H 3050 5200 50  0000 L CNN
-F 2 "" V 2950 5260 50  0001 C CNN
+F 2 "spang_badge:COINCELL_20MM" V 2950 5260 50  0001 C CNN
 F 3 "" V 2950 5260 50  0000 C CNN
 	1    2950 5200

Commit message: routing sponge. Need to figure out how to rename polygons to GND
Parts:
- removed D6, D7: LED, LEDs:LED_0603, symbol LED
- removed P1: PROGRAM, symbol CONN_01X05
- removed R1, R2, R3, R4, R5, R6, R7: R, Resistors_SMD:R_0603, symbol R
- removed SW1: SW_DPST, Buttons_Switches_SMD:SW_SPST_EVQPE1, symbol SW_DPST
- added J1: CONN-TAGCONNECT-TC2050, spang_badge:TC2050_IDC, symbol CONN-TAGCONNECT-TC2050
- added SW1: SW_SPST, Buttons_Switches_SMD:SW_SPST_B3U-3000P, symbol SW_SPST
- Q1: footprint (none) -> TO_SOT_Packages_SMD:SOT-23
- renumbered D8 to D7, D9 to D8, R8 to R1, R9 to R2
Connections:
- net labels added: TCK, TDI, nRST
- net labels removed: BACKLIGHT
- wire segments 58 -> 53
Other:
- moved on the sheet: BT1, D1, D2, D3, D4, D5, D7, D8, F1, IC1, R1, R2

Commit message: need to run DRC
Parts:
- SW1: footprint Buttons_Switches_SMD:SW_SPST_B3U-3000P -> spang_badge:EVQ-P7B01P
Changed lines of the file:
@@
 F 0 "SW1" H 6300 4325 50  0000 C CNN
 F 1 "SW_SPST" H 6300 4100 50  0000 C CNN
-F 2 "Buttons_Switches_SMD:SW_SPST_B3U-3000P" H 6300 4200 50  0001 C CNN
+F 2 "spang_badge:EVQ-P7B01P" H 6300 4200 50  0001 C CNN
 F 3 "" H 6300 4200 50  0001 C CNN
 	1    6300 4200
@@
 Connection ~ 6800 5650
 $Comp
-L +BATT #PWR?
+L +BATT #PWR010
 U 1 1 5D5FB127
 P 5800 5450
-F 0 "#PWR?" H 5800 5300 50  0001 C CNN
+F 0 "#PWR010" H 5800 5300 50  0001 C CNN
 F 1 "+BATT" H 5800 5590 50  0000 C CNN
 F 2 "" H 5800 5450 50  0001 C CNN
@@
 $EndComp
 $Comp
-L GND #PWR?
+L GND #PWR011
 U 1 1 5D5FB15F
 P 5800 5650
-F 0 "#PWR?" H 5800 5400 50  0001 C CNN
+F 0 "#PWR011" H 5800 5400 50  0001 C CNN
 F 1 "GND" H 5800 5500 50  0000 C CNN
 F 2 "" H 5800 5650 50  0000 C CNN
@@
 $EndComp
 $Comp
-L GND #PWR?
+L GND #PWR012
 U 1 1 5D5FB197
 P 5800 5850
-F 0 "#PWR?" H 5800 5600 50  0001 C CNN
+F 0 "#PWR012" H 5800 5600 50  0001 C CNN
 F 1 "GND" H 5800 5700 50  0000 C CNN
 F 2 "" H 5800 5850 50  0000 C CNN
@@
 $EndComp
 $Comp
-L GND #PWR?
+L GND #PWR013
 U 1 1 5D5FB1CF
 P 6800 5550
-F 0 "#PWR?" H 6800 5300 50  0001 C CNN
+F 0 "#PWR013" H 6800 5300 50  0001 C CNN
 F 1 "GND" H 6800 5400 50  0000 C CNN
 F 2 "" H 6800 5550 50  0000 C CNN

Commit message: working on spang badge v2. TODO: fix B-CU
Parts:
- J1: footprint spang_badge:TC2050_IDC -> spang_badge:TC2050-All_Holes
- R1, R2: footprint Resistors_SMD:R_0603 -> Resistors_SMD:R_0603_HandSoldering
Changed lines of the file:
@@
 F 0 "R1" H 9780 4100 50  0000 C CNN
 F 1 "R" V 9700 4100 50  0000 C CNN
-F 2 "Resistors_SMD:R_0603" V 9630 4100 50  0001 C CNN
+F 2 "Resistors_SMD:R_0603_HandSoldering" V 9630 4100 50  0001 C CNN
 F 3 "" H 9700 4100 50  0000 C CNN
 	1    9700 4100
@@
 F 0 "R2" V 10080 4100 50  0000 C CNN
 F 1 "R" V 10000 4100 50  0000 C CNN
-F 2 "Resistors_SMD:R_0603" V 9930 4100 50  0001 C CNN
+F 2 "Resistors_SMD:R_0603_HandSoldering" V 9930 4100 50  0001 C CNN
 F 3 "" H 10000 4100 50  0000 C CNN
 	1    10000 4100
@@
 F 0 "J1" H 6300 6100 50  0000 C CNN
 F 1 "CONN-TAGCONNECT-TC2050" H 6300 6000 50  0000 C CNN
-F 2 "spang_badge:TC2050_IDC" H 6150 5850 50  0001 C CNN
+F 2 "spang_badge:TC2050-All_Holes" H 6150 5850 50  0001 C CNN
 F 3 "" H 6150 5850 50  0000 C CNN
 	1    6300 5650

Commit message: workin on cryptid shroom
Connections:
- wire segments 53 -> 51
Changed lines of the file:
@@
 	6100 5750 5800 5750
-Wire Wire Line
-	6500 5650 6800 5650
-Wire Wire Line
-	6500 5450 6800 5450
 Wire Wire Line
 	6100 5650 5800 5650
 Wire Wire Line
-	6100 5850 5800 5850
+	6100 5450 5800 5450
 Wire Wire Line
-	6500 5550 6800 5550
+	6100 5550 5800 5550
+Text Label 5800 5450 0    60   ~ 0
+TCK
+Text Label 5800 5650 0    60   ~ 0
+TDI
 Wire Wire Line
-	6100 5450 5800 5450
-Connection ~ 5800 5750
-Connection ~ 6800 5450
-Connection ~ 6800 5650
+	6500 5850 6800 5850
+Text Label 6800 5850 2    60   ~ 0
+nRST
 $Comp
-L +BATT #PWR010
-U 1 1 5D5FB127
-P 5800 5450
-F 0 "#PWR010" H 5800 5300 50  0001 C CNN
-F 1 "+BATT" H 5800 5590 50  0000 C CNN
-F 2 "" H 5800 5450 50  0001 C CNN
-F 3 "" H 5800 5450 50  0001 C CNN
-	1    5800 5450
-	0    -1   -1   0
-$EndComp
-$Comp
-L GND #PWR011
-U 1 1 5D5FB15F
-P 5800 5650
-F 0 "#PWR011" H 5800 5400 50  0001 C CNN
-F 1 "GND" H 5800 5500 50  0000 C CNN
-F 2 "" H 5800 5650 50  0000 C CNN
-F 3 "" H 5800 5650 50  0000 C CNN
-	1    5800 5650
+L GND #PWR?
+U 1 1 5D871F42
+P 5800 5550
+F 0 "#PWR?" H 5800 5300 50  0001 C CNN
+F 1 "GND" H 5800 5400 50  0000 C CNN
+F 2 "" H 5800 5550 50  0000 C CNN
+F 3 "" H 5800 5550 50  0000 C CNN
+	1    5800 5550
 	0    1    1    0
 $EndComp
 $Comp
-L GND #PWR012
-U 1 1 5D5FB197
-P 5800 5850
-F 0 "#PWR012" H 5800 5600 50  0001 C CNN
-F 1 "GND" H 5800 5700 50  0000 C CNN
-F 2 "" H 5800 5850 50  0000 C CNN
-F 3 "" H 5800 5850 50  0000 C CNN
-	1    5800 5850
-	0    1    1    0
-$EndComp
-$Comp
-L GND #PWR013
-U 1 1 5D5FB1CF
-P 6800 5550
-F 0 "#PWR013" H 6800 5300 50  0001 C CNN
-F 1 "GND" H 6800 5400 50  0000 C CNN
-F 2 "" H 6800 5550 50  0000 C CNN
-F 3 "" H 6800 5550 50  0000 C CNN
-	1    6800 5550
+L +BATT #PWR?
+U 1 1 5D8721F0
+P 5800 5750
+F 0 "#PWR?" H 5800 5600 50  0001 C CNN
+F 1 "+BATT" H 5800 5890 50  0000 C CNN
+F 2 "" H 5800 5750 50  0001 C CNN
+F 3 "" H 5800 5750 50  0001 C CNN
+	1    5800 5750
 	0    -1   -1   0
 $EndComp
-Text Label 6000 5750 2    60   ~ 0
-TCK
-Text Label 6700 5650 0    60   ~ 0
-TDI
-Text Label 6800 5450 0    60   ~ 0
-nRST
 $EndSCHEMATC
