File: board-kicad/vineshroom_badge-corrupted.kicad_pcb (KiCad board)
At the start: 2 copper layers, 95 x 95.7 mm, 78 parts, among them IC1 ATTINY20-X, J1 CONN-TAGCONNECT-TC2050, Q1 Q_NMOS_DGS, SW1 SW_SPST

Commit message: workin on cryptid shroom
Parts:
- removed the G*** at (140.5, 94.0)
- added G***: LOGO, vine_badge:VINESHROOM_CORRUPTED_SILKSCREEN, F.Cu at (140.7, 93.7)
- moved D1 35.6 mm to (141.5, 128.4), turned to 270 degrees
- moved D10 32.6 mm to (132.8, 128.5), turned to 90 degrees
- moved D13 31.5 mm to (126.5, 126.2), turned to 45 degrees
- moved D8 30.3 mm to (141.0, 125.5), turned to 270 degrees
- moved D11 26.6 mm to (132.1, 125.5), turned to 270 degrees
- moved D6 25.3 mm to (128.8, 123.9), turned to 45 degrees
- moved D2 25.2 mm to (140.5, 122.4), turned to 90 degrees
- moved D4 20.6 mm to (131.6, 122.4), turned to 270 degrees
- moved D9 20.5 mm to (139.9, 119.3), turned to 270 degrees
- moved D7 19.4 mm to (128.3, 120.4), turned to 315 degrees
- moved D14 19.2 mm to (125.7, 117.9), turned to 315 degrees
- moved D3 17.1 mm to (139.7, 116.1), turned to 90 degrees
- moved D5 14.6 mm to (131.1, 119.4), turned to 270 degrees
- moved D12 8.83 mm to (130.5, 116.2), turned to 270 degrees
Routing:
- net Net-(D10-Pad1): track 189.0 -> 135.1 mm, vias 8 -> 6
- net Net-(D1-Pad1): track 105.0 -> 74.3 mm, vias 3 -> 1
- net Net-(D10-Pad2): track 150.4 -> 121.1 mm, vias 4 -> 2
- net /BTN: track 50.7 -> 26.6 mm, vias 2 -> 0
- net Net-(D11-Pad2): track 103.8 -> 83.7 mm, vias 10 -> 8
- net Net-(D13-Pad2): track 143.2 -> 125.3 mm, vias 7 -> 5
- net Net-(D12-Pad2): track 137.2 -> 120.1 mm, vias 12 -> 10
- net Net-(D1-Pad2): track 143.9 -> 134.5 mm, vias 7 -> 6
- net Net-(D14-Pad2): track 134.0 -> 125.8 mm, vias 4 -> 3
- net (no net): track 0.00 -> 1.93 mm
Other:
- board text removed: "JLCJLCJLCJLC"
