File: board-kicad/VineBadge2020.sch (KiCad schematic (older format))
At the start: 71 parts, among them IC1 ATTINY20-X, J1 CONN-TAGCONNECT-TC2050, Q1 Q_NMOS_DGS, SW1 SW_SPST, SW2 SW_DPDT_x2

Commit message: fixed pinout on programming header, some other shit too whatever lets get this done
Parts:
- removed Q1: Q_NMOS_DGS, TO_SOT_Packages_SMD:SOT-23, symbol Q_NMOS_DGS
- removed R1, R2, R3, R4, R5, R6, R7, R8: R, Resistors_SMD:R_0805, symbol R
- added D53: D_Schottky, Diodes_SMD:SOD-323_HandSoldering, symbol D_Schottky
- added TP_BATT1, TP_GND1: TEST, Pin_Headers:Pin_Header_Straight_1x01, symbol TEST
- C1, C2: footprint Capacitors_SMD:C_0603 -> Capacitors_SMD:C_0805_HandSoldering
- D1: LCSC (none) -> C205443
- J1: footprint vine_badge:TC2050_IDC -> vine_badge:TC2050-All_Holes
- R10, R9: footprint Resistors_SMD:R_0805 -> Resistors_SMD:R_0805_HandSoldering
- renumbered SW2 to ON/OFF1
Connections:
- net +BATT: now also J1.7, D53.1 (K); no longer F1.1, J1.4
- net GND: now also BT1.2 (-), J1.9, TP_GND1.1; no longer J1.2
- net RST: now also J1.5; no longer J1.6
- net TCK: now also J1.10; no longer J1.1
- net TDI: now also J1.8; no longer J1.3
- net at IC1.10 ((PCINT3/ADC3)PA3): now also D10.2 (A), D11.1 (K), D17.1 (K), D18.2 (A), D21.1 (K), D22.2 (A), D23.2 (A), D24.1 (K), D3.1 (K), D33.2 (A), D34.1 (K), D4.2 (A), D43.2 (A), D44.1 (K)
- net at IC1.11 ((PCINT2/AIN1/ADC2)PA2): now also D10.1 (K), D15.1 (K), D16.2 (A), D19.2 (A), D2.1 (K), D20.1 (K), D29.2 (A), D3.2 (A), D31.1 (K), D41.2 (A), D42.1 (K), D49.2 (A), D50.2 (A), D9.2 (A)
- net at IC1.12 ((PCINT1/AIN0/ADC1)PA1): now also D1.1 (K), D17.2 (A), D18.1 (K), D2.2 (A), D25.2 (A), D27.1 (K), D39.2 (A), D40.1 (K), D8.2 (A), D9.1 (K)
- net at IC1.13 ((PCINT0/ADC0)PA0): now also D1.2 (A), D15.2 (A), D16.1 (K), D21.2 (A), D23.1 (K), D35.2 (A), D37.1 (K), D45.2 (A), D46.1 (K), D47.2 (A), D48.1 (K), D51.2 (A), D52.1 (K), D8.1 (K)
- net at IC1.6 ((PCINT7/SCL/SCK/T1/ICP1/OC0B/ADC7)PA7): now also D14.2 (A), D30.1 (K), D32.2 (A), D36.1 (K), D38.2 (A), D43.1 (K), D44.2 (A), D49.1 (K), D50.1 (K), D7.1 (K)
- net at IC1.7 ((PCINT6/~SS~/ADC6)PA6): now also D13.2 (A), D14.1 (K), D26.1 (K), D28.2 (A), D33.1 (K), D34.2 (A), D41.1 (K), D42.2 (A), D47.1 (K), D48.2 (A), D51.1 (K), D52.2 (A), D6.1 (K), D7.2 (A)
- net at IC1.8 ((PCINT5/ADC5)PA5): now also D12.2 (A), D13.1 (K), D22.1 (K), D24.2 (A), D29.1 (K), D30.2 (A), D31.2 (A), D32.1 (K), D39.1 (K), D40.2 (A), D45.1 (K), D46.2 (A), D5.1 (K), D6.2 (A)
- net at IC1.9 ((PCINT4/ADC4)PA4): now also D11.2 (A), D12.1 (K), D19.1 (K), D20.2 (A), D25.1 (K), D26.2 (A), D27.2 (A), D28.1 (K), D35.1 (K), D36.2 (A), D37.2 (A), D38.1 (K), D4.1 (K), D5.2 (A)
- net at BT1.1 (+), ON/OFF1.2 (B): now also TP_BATT1.1
- new net: D53.2 (A), F1.1
Changed lines of the file:
@@
 	1    0    0    -1
-$EndComp
-$Comp
-L R R1
-U 1 1 5D1D4171
-P 6550 1500
-F 0 "R1" V 6630 1500 50  0000 C CNN
-F 1 "R" V 6550 1500 50  0000 C CNN
-F 2 "Resistors_SMD:R_0805" V 6480 1500 50  0001 C CNN
-F 3 "" H 6550 1500 50  0000 C CNN
-	1    6550 1500
-	0    1    1    0
-$EndComp
-$Comp
-L R R2
-U 1 1 5D1D437F
-P 6550 1700
-F 0 "R2" V 6630 1700 50  0000 C CNN
-F 1 "R" V 6550 1700 50  0000 C CNN
-F 2 "Resistors_SMD:R_0805" V 6480 1700 50  0001 C CNN
-F 3 "" H 6550 1700 50  0000 C CNN
-	1    6550 1700
-	0    1    1    0
-$EndComp
-$Comp
-L R R3
-U 1 1 5D1D43C2
-P 6550 1900
-F 0 "R3" V 6630 1900 50  0000 C CNN
-F 1 "R" V 6550 1900 50  0000 C CNN
-F 2 "Resistors_SMD:R_0805" V 6480 1900 50  0001 C CNN
-F 3 "" H 6550 1900 50  0000 C CNN
-	1    6550 1900
-	0    1    1    0
-$EndComp
-$Comp
-L R R4
-U 1 1 5D1D4409
-P 6550 2100
-F 0 "R4" V 6630 2100 50  0000 C CNN
-F 1 "R" V 6550 2100 50  0000 C CNN
-F 2 "Resistors_SMD:R_0805" V 6480 2100 50  0001 C CNN
-F 3 "" H 6550 2100 50  0000 C CNN
-	1    6550 2100
-	0    1    1    0
-$EndComp
-$Comp
-L R R5
-U 1 1 5D1D446B
-P 6550 2300
-F 0 "R5" V 6630 2300 50  0000 C CNN
-F 1 "R" V 6550 2300 50  0000 C CNN
-F 2 "Resistors_SMD:R_0805" V 6480 2300 50  0001 C CNN
-F 3 "" H 6550 2300 50  0000 C CNN
-	1    6550 2300
-	0    1    1    0
-$EndComp
-$Comp
-L R R6
-U 1 1 5D1D44DE
-P 6550 2500
-F 0 "R6" V 6630 2500 50  0000 C CNN
-F 1 "R" V 6550 2500 50  0000 C CNN
-F 2 "Resistors_SMD:R_0805" V 6480 2500 50  0001 C CNN
-F 3 "" H 6550 2500 50  0000 C CNN
-	1    6550 2500
-	0    1    1    0
-$EndComp
-$Comp
-L R R7
-U 1 1 5D1D4559
-P 6550 2700
-F 0 "R7" V 6630 2700 50  0000 C CNN
-F 1 "R" V 6550 2700 50  0000 C CNN
-F 2 "Resistors_SMD:R_0805" V 6480 2700 50  0001 C CNN
-F 3 "" H 6550 2700 50  0000 C CNN
-	1    6550 2700
-	0    1    1    0
-$EndComp
-$Comp
-L R R8
-U 1 1 5D1D45D2
-P 6550 2900
-F 0 "R8" V 6630 2900 50  0000 C CNN
-F 1 "R" V 6550 2900 50  0000 C CNN
-F 2 "Resistors_SMD:R_0805" V 6480 2900 50  0001 C CNN
-F 3 "" H 6550 2900 50  0000 C CNN
-	1    6550 2900
-	0    1    1    0
 $EndComp
 Text Label 4450 2400 0    60   ~ 0
@@
 F 2 "LEDs:LED_0603" H 7250 1650 50  0001 C CNN
 F 3 "" H 7250 1650 50  0000 C CNN
+F 4 "C205443" H 7250 1650 60  0001 C CNN "LCSC"
 	1    7250 1650
 	0    -1   -1   0
@@
 $EndComp
 $Comp
-L Q_NMOS_DGS Q1
-U 1 1 5D2359E3
-P 3500 3550
-F 0 "Q1" H 3700 3600 50  0000 L CNN
-F 1 "Q_NMOS_DGS" H 3700 3500 50  0000 L CNN
-F 2 "TO_SOT_Packages_SMD:SOT-23" H 3700 3650 50  0001 C CNN
-F 3 "" H 3500 3550 50  0000 C CNN
-	1    3500 3550
-	0    -1   1    0
-$EndComp
-$Comp
 L GND #PWR03
 U 1 1 5D236972
@@
 F 0 "R9" V 4780 2900 50  0000 C CNN
 F 1 "1K" V 4700 2900 50  0000 C CNN
-F 2 "Resistors_SMD:R_0805" V 4630 2900 50  0001 C CNN
+F 2 "Resistors_SMD:R_0805_HandSoldering" V 4630 2900 50  0001 C CNN
 F 3 "" H 4700 2900 50  0000 C CNN
 	1    4700 2900
@@
 F 0 "C1" H 2075 1800 50  0000 L CNN
 F 1 "100nF" H 2075 1600 50  0000 L CNN
-F 2 "Capacitors_SMD:C_0603" H 2088 1550 50  0001 C CNN
+F 2 "Capacitors_SMD:C_0805_HandSoldering" H 2088 1550 50  0001 C CNN
 F 3 "" H 2050 1700 50  0000 C CNN
 	1    2050 1700
@@
 F 0 "J1" H 5550 4450 50  0000 C CNN
 F 1 "CONN-TAGCONNECT-TC2050" H 5550 4350 50  0000 C CNN
-F 2 "vine_badge:TC2050_IDC" H 5400 4200 50  0001 C CNN
+F 2 "vine_badge:TC2050-All_Holes" H 5400 4200 50  0001 C CNN
 F 3 "" H 5400 4200 50  0000 C CNN
 	1    5550 4000
@@
 	-1   0    0    1
 $EndComp
-Text Label 6000 4200 0    60   ~ 0
-RST
 $Comp
 L SW_SPST SW1
@@
 $EndComp
 $Comp
-L GND #PWR011
+L GND #PWR07
 U 1 1 5D63930F
 P 3400 5050
-F 0 "#PWR011" H 3400 4800 50  0001 C CNN
+F 0 "#PWR07" H 3400 4800 50  0001 C CNN
 F 1 "GND" H 3400 4900 50  0000 C CNN
 F 2 "" H 3400 5050 50  0000 C CNN
@@
 F 0 "R10" V 2780 4650 50  0000 C CNN
 F 1 "1K" V 2700 4650 50  0000 C CNN
-F 2 "Resistors_SMD:R_0805" V 2630 4650 50  0001 C CNN
+F 2 "Resistors_SMD:R_0805_HandSoldering" V 2630 4650 50  0001 C CNN
 F 3 "" H 2700 4650 50  0000 C CNN
 	1    2700 4650
@@
 $EndComp
 $Comp
-L +BATT #PWR012
+L +BATT #PWR08
 U 1 1 5D63FB11
 P 2700 4450
-F 0 "#PWR012" H 2700 4300 50  0001 C CNN
+F 0 "#PWR08" H 2700 4300 50  0001 C CNN
 F 1 "+BATT" H 2700 4590 50  0000 C CNN
 F 2 "" H 2700 4450 50  0000 C CNN
@@
 $EndComp
 $Comp
-L SW_DPDT_x2 SW2
+L SW_DPDT_x2 ON/OFF1
 U 1 1 5D63860F
 P 2350 3250
-F 0 "SW2" H 2350 3420 50  0000 C CNN
+F 0 "ON/OFF1" H 2350 3420 50  0000 C CNN
 F 1 "SW_DPDT_x2" H 2350 3050 50  0000 C CNN
 F 2 "vine_badge:JS202011JAQN" H 2350 3250 50  0001 C CNN
@@
 	2050 2750 2050 2700
 Wire Wire Line
-	4450 1500 6400 1500
+	4450 1500 17750 1500
 Wire Wire Line
 	4450 1600 6400 1600
@@
 	6350 1700 6350 1900
 Wire Wire Line
-	6350 1900 6400 1900
+	6350 1900 7100 1900
 Wire Wire Line
 	4450 1800 6300 1800
@@
 	6300 1800 6300 2100
 Wire Wire Line
-	6300 2100 6400 2100
+	6300 2100 7050 2100
 Wire Wire Line
 	4450 1900 6250 1900
@@
 	6250 1900 6250 2300
 Wire Wire Line
-	6250 2300 6400 2300
+	6250 2300 7000 2300
 Wire Wire Line
 	4450 2000 6200 2000
@@
 	6200 2000 6200 2500
 Wire Wire Line
-	6200 2500 6400 2500
+	6200 2500 6950 2500
 Wire Wire Line
 	4450 2100 6150 2100
@@
 	6150 2100 6150 2700
 Wire Wire Line
-	6150 2700 6400 2700
+	6150 2700 6900 2700
 Wire Wire Line
 	4450 2200 6100 2200
@@
 	6100 2200 6100 2900
 Wire Wire Line
-	6100 2900 6400 2900
+	6100 2900 6850 2900
 Wire Wire Line
 	4450 2400 5300 2400
@@
 Connection ~ 7250 1500
 Wire Wire Line
-	6700 1700 7150 1700
+	6400 1700 7150 1700
 Wire Wire Line
 	7150 1700 7150 1850
@@
 Connection ~ 7250 1850
 Wire Wire Line
-	6700 1900 7100 1900
-Wire Wire Line
 	7100 1900 7100 2250
 Wire Wire Line
@@
 Connection ~ 7250 2250
 Wire Wire Line
-	6700 2100 7050 2100
-Wire Wire Line
 	7050 2100 7050 2650
 Wire Wire Line
@@
 Connection ~ 7250 2650
 Wire Wire Line
-	6700 2300 7000 2300
-Wire Wire Line
 	7000 2300 7000 3050
 Wire Wire Line
@@
 Connection ~ 7250 3050
 Wire Wire Line
-	6700 2500 6950 2500
-Wire Wire Line
 	6950 2500 6950 3450
 Wire Wire Line
@@
 Connection ~ 7250 3450
 Wire Wire Line
-	6700 2700 6900 2700
-Wire Wire Line
 	6900 2700 6900 3850
 Wire Wire Line
 	7250 3800 7250 3900
 Connection ~ 7250 3850
-Wire Wire Line
-	6700 2900 6850 2900
 Wire Wire Line
 	6850 2900 6850 4200
@@
 	16550 3850 16550 3800
 Connection ~ 16550 3850
-Wire Wire Line
-	6700 1500 17750 1500
 Connection ~ 7550 1500
 Wire Wire Line
@@
 Connection ~ 7550 4200
 Wire Wire Line
-	1650 3650 3300 3650
-Connection ~ 3500 3350
-Wire Wire Line
-	3700 3650 4050 3650
+	1650 3650 4050 3650
 Wire Wire Line
 	4050 3650 4050 3700
-Wire Wire Line
-	3150 3350 4050 3350
-Wire Wire Line
-	3500 3350 3850 3350
 Connection ~ 3850 3350
 Connection ~ 3850 3650
@@
 Connection ~ 5300 2500
 Connection ~ 5300 2600
-Wire Wire Line
-	5350 3800 4950 3800
-Wire Wire Line
-	5350 4000 4950 4000
-Wire Wire Line
-	4950 4100 5350 4100
 Wire Wire Line
 	2400 4850 2700 4850
@@
 F 0 "C2" H 3875 3600 50  0000 L CNN
 F 1 "1uF" H 3875 3400 50  0000 L CNN
-F 2 "Capacitors_SMD:C_0603" H 3888 3350 50  0001 C CNN
+F 2 "Capacitors_SMD:C_0805_HandSoldering" H 3888 3350 50  0001 C CNN
 F 3 "" H 3850 3500 50  0000 C CNN
 	1    3850 3500
 	1    0    0    -1
 $EndComp
-Text Label 4950 3800 0    60   ~ 0
+Wire Wire Line
+	5750 3800 6150 3800
+Wire Wire Line
+	5750 3900 6150 3900
+Wire Wire Line
+	5750 4000 6150 4000
+Wire Wire Line
+	5750 4100 6150 4100
+Wire Wire Line
+	5350 4200 4900 4200
+Text Label 4900 4200 0    60   ~ 0
+RST
+Text Label 6150 3800 2    60   ~ 0
 TCK
-Text Label 4950 4000 0    60   ~ 0
+Text Label 6150 4000 2    60   ~ 0
 TDI
-Wire Wire Line
-	6150 4200 5750 4200
-Connection ~ 6150 4200
-Wire Wire Line
-	5350 3900 4950 3900
-Connection ~ 4950 4000
-Connection ~ 4950 3800
-$Comp
-L +BATT #PWR?
-U 1 1 5D874440
-P 4950 4100
-F 0 "#PWR?" H 4950 3950 50  0001 C CNN
-F 1 "+BATT" H 4950 4240 50  0000 C CNN
-F 2 "" H 4950 4100 50  0000 C CNN
-F 3 "" H 4950 4100 50  0000 C CNN
-	1    4950 4100
-	0    -1   -1   0
-$EndComp
-$Comp
-L GND #PWR?
-U 1 1 5D8784AD
-P 4950 3900
-F 0 "#PWR?" H 4950 3650 50  0001 C CNN
-F 1 "GND" H 4950 3750 50  0000 C CNN
-F 2 "" H 4950 3900 50  0000 C CNN
-F 3 "" H 4950 3900 50  0000 C CNN
-	1    4950 3900
-	0    1    1    0
+$Comp
+L GND #PWR09
+U 1 1 5DD8F695
+P 6150 3900
+F 0 "#PWR09" H 6150 3650 50  0001 C CNN
+F 1 "GND" H 6150 3750 50  0000 C CNN
+F 2 "" H 6150 3900 50  0000 C CNN
+F 3 "" H 6150 3900 50  0000 C CNN
+	1    6150 3900
+	0    -1   -1   0
+$EndComp
+$Comp
+L +BATT #PWR010
+U 1 1 5DD8F89B
+P 6150 4100
+F 0 "#PWR010" H 6150 3950 50  0001 C CNN
+F 1 "+BATT" H 6150 4240 50  0000 C CNN
+F 2 "" H 6150 4100 50  0000 C CNN
+F 3 "" H 6150 4100 50  0000 C CNN
+	1    6150 4100
+	0    1    1    0
+$EndComp
+Connection ~ 6150 3800
+Connection ~ 6150 4000
+Connection ~ 4900 4200
+$Comp
+L D_Schottky D53
+U 1 1 5DDA5070
+P 3500 3350
+F 0 "D53" H 3500 3450 50  0000 C CNN
+F 1 "D_Schottky" H 3500 3250 50  0000 C CNN
+F 2 "Diodes_SMD:SOD-323_HandSoldering" H 3500 3350 50  0001 C CNN
+F 3 "" H 3500 3350 50  0000 C CNN
+	1    3500 3350
+	-1   0    0    1
+$EndComp
+Wire Wire Line
+	3650 3350 4050 3350
+Wire Wire Line
+	3350 3350 3150 3350
+$Comp
+L TEST TP_BATT1
+U 1 1 5DDB3DBD
+P 1650 3250
+F 0 "TP_BATT1" H 1650 3550 50  0000 C BNN
+F 1 "TEST" H 1650 3500 50  0000 C CNN
+F 2 "Pin_Headers:Pin_Header_Straight_1x01" H 1650 3250 50  0001 C CNN
+F 3 "" H 1650 3250 50  0000 C CNN
+	1    1650 3250
+	1    0    0    -1
+$EndComp
+$Comp
+L TEST TP_GND1
+U 1 1 5DDB472A
+P 1650 3650
+F 0 "TP_GND1" H 1650 3950 50  0000 C BNN
+F 1 "TEST" H 1650 3900 50  0000 C CNN
+F 2 "Pin_Headers:Pin_Header_Straight_1x01" H 1650 3650 50  0001 C CNN
+F 3 "" H 1650 3650 50  0000 C CNN
+	1    1650 3650
+	-1   0    0    1
 $EndComp
 $EndSCHEMATC
