File: board/Shroom/VineBadge2020.sch (KiCad schematic (older format))
At the start: 66 parts, among them IC1 ATTINY20-X, J1 CONN-TAGCONNECT-TC2050, SW1 SW_SPDT, SW2 SW_Push

Commit message: created a progmem led map, need ot test
Parts:
- renumbered D53 to D57
Connections:
- net at D10.1 (K), D15.1 (K), D16.2 (A)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: now also D50.1 (K); no longer D50.2 (A)
- net at D14.2 (A), D30.1 (K), D32.2 (A)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: now also D50.2 (A), D51.1 (K), D52.2 (A); no longer D50.1 (K)
- net at D13.2 (A), D14.1 (K), D26.1 (K)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: no longer D51.1 (K), D52.2 (A)
Other:
- moved on the sheet: D50

Commit message: removed programming stuff, getting ready for final revision. Just needs last checks
Parts:
- removed C1: 100nF, Capacitors_SMD:C_0805_HandSoldering, symbol C
- removed C2: 1uF, Capacitors_SMD:C_0805_HandSoldering, symbol C
- removed J1: CONN-TAGCONNECT-TC2050, VineBadge2020:TC2050-All_Holes, symbol CONN-TAGCONNECT-TC2050
- removed R10: 1K, Resistors_SMD:R_0805_HandSoldering, symbol R
- removed SW1: SW_SPDT, VineBadge2020:JS202011JAQN-Handsolder, symbol SW_SPDT
- SW2: footprint VineBadge2020:SW_SPST_EVQPE1_Handsolder -> Buttons_Switches_SMD:SW_SPST_TL3342
Connections:
- net GND: now also F1.1; no longer BT1.2 (-)
- net at BT1.1 (+): now also D57.2 (A)
- net at F1.2: now also BT1.2 (-)
Other:
- moved on the sheet: BT1, F1
Changed lines of the file:
@@
 L Battery_Cell BT1
 U 1 1 5D2356C4
-P 1650 3550
-F 0 "BT1" H 1750 3650 50  0000 L CNN
-F 1 "Battery_Cell" H 1750 3550 50  0000 L CNN
-F 2 "VineBadge2020:COINCELL_20MM_HANDSOLDER" V 1650 3610 50  0001 C CNN
-F 3 "" V 1650 3610 50  0000 C CNN
-	1    1650 3550
+P 3050 3650
+F 0 "BT1" H 3150 3750 50  0000 L CNN
+F 1 "Battery_Cell" H 3150 3650 50  0000 L CNN
+F 2 "VineBadge2020:COINCELL_20MM_HANDSOLDER" V 3050 3710 50  0001 C CNN
+F 3 "" V 3050 3710 50  0000 C CNN
+	1    3050 3650
 	1    0    0    -1
 $EndComp
@@
 L GND #PWR03
 U 1 1 5D236972
-P 4050 3700
-F 0 "#PWR03" H 4050 3450 50  0001 C CNN
-F 1 "GND" H 4050 3550 50  0000 C CNN
-F 2 "" H 4050 3700 50  0000 C CNN
-F 3 "" H 4050 3700 50  0000 C CNN
-	1    4050 3700
+P 3850 3900
+F 0 "#PWR03" H 3850 3650 50  0001 C CNN
+F 1 "GND" H 3850 3750 50  0000 C CNN
+F 2 "" H 3850 3900 50  0000 C CNN
+F 3 "" H 3850 3900 50  0000 C CNN
+	1    3850 3900
 	1    0    0    -1
 $EndComp
@@
 L +BATT #PWR04
 U 1 1 5D236A0E
-P 4050 3350
-F 0 "#PWR04" H 4050 3200 50  0001 C CNN
-F 1 "+BATT" H 4050 3490 50  0000 C CNN
-F 2 "" H 4050 3350 50  0000 C CNN
-F 3 "" H 4050 3350 50  0000 C CNN
-	1    4050 3350
+P 3850 3350
+F 0 "#PWR04" H 3850 3200 50  0001 C CNN
+F 1 "+BATT" H 3850 3490 50  0000 C CNN
+F 2 "" H 3850 3350 50  0000 C CNN
+F 3 "" H 3850 3350 50  0000 C CNN
+	1    3850 3350
 	1    0    0    -1
 $EndComp
@@
 L Fuse F1
 U 1 1 5D237CDD
-P 3000 3350
-F 0 "F1" V 3080 3350 50  0000 C CNN
-F 1 "Fuse" V 2925 3350 50  0000 C CNN
-F 2 "Fuse_Holders_and_Fuses:Fuse_SMD1206_Reflow" V 2930 3350 50  0001 C CNN
-F 3 "" H 3000 3350 50  0000 C CNN
-	1    3000 3350
+P 3500 3850
+F 0 "F1" V 3600 3850 50  0000 C CNN
+F 1 "Fuse" V 3425 3850 50  0000 C CNN
+F 2 "Fuse_Holders_and_Fuses:Fuse_SMD1206_Reflow" V 3430 3850 50  0001 C CNN
+F 3 "" H 3500 3850 50  0000 C CNN
+	1    3500 3850
 	0    1    1    0
 $EndComp
@@
 	1    0    0    -1
 $EndComp
-$Comp
-L C C1
-U 1 1 5D239B6F
-P 2050 1700
-F 0 "C1" H 2075 1800 50  0000 L CNN
-F 1 "100nF" H 2075 1600 50  0000 L CNN
-F 2 "Capacitors_SMD:C_0805_HandSoldering" H 2088 1550 50  0001 C CNN
-F 3 "" H 2050 1700 50  0000 C CNN
-	1    2050 1700
-	1    0    0    -1
-$EndComp
-$Comp
-L GND #PWR05
-U 1 1 5D239DAF
-P 2050 1900
-F 0 "#PWR05" H 2050 1650 50  0001 C CNN
-F 1 "GND" H 2050 1750 50  0000 C CNN
-F 2 "" H 2050 1900 50  0000 C CNN
-F 3 "" H 2050 1900 50  0000 C CNN
-	1    2050 1900
-	1    0    0    -1
-$EndComp
 Text Notes 15350 5550 0    60   ~ 12
 Vinesauce TMG 2020 Badge
@@
 0.3
 $Comp
-L CONN-TAGCONNECT-TC2050 J1
-U 1 1 5D6340F6
-P 5550 4000
-F 0 "J1" H 5550 4450 50  0000 C CNN
-F 1 "CONN-TAGCONNECT-TC2050" H 5550 4350 50  0000 C CNN
-F 2 "VineBadge2020:TC2050-All_Holes" H 5400 4200 50  0001 C CNN
-F 3 "" H 5400 4200 50  0000 C CNN
-	1    5550 4000
-	1    0    0    -1
-$EndComp
-$Comp
-L +BATT #PWR06
+L +BATT #PWR05
 U 1 1 5D1D5CCC
 P 4700 3100
-F 0 "#PWR06" H 4700 2950 50  0001 C CNN
+F 0 "#PWR05" H 4700 2950 50  0001 C CNN
 F 1 "+BATT" H 4700 3240 50  0000 C CNN
 F 2 "" H 4700 3100 50  0000 C CNN
@@
 $EndComp
 $Comp
-L GND #PWR07
+L GND #PWR06
 U 1 1 5D63930F
 P 3400 5050
-F 0 "#PWR07" H 3400 4800 50  0001 C CNN
+F 0 "#PWR06" H 3400 4800 50  0001 C CNN
 F 1 "GND" H 3400 4900 50  0000 C CNN
 F 2 "" H 3400 5050 50  0000 C CNN
@@
 Text Label 2400 4850 0    60   ~ 0
 BTN
-$Comp
-L R R10
-U 1 1 5D63DC4D
-P 2700 4650
-F 0 "R10" V 2780 4650 50  0000 C CNN
-F 1 "1K" V 2700 4650 50  0000 C CNN
-F 2 "Resistors_SMD:R_0805_HandSoldering" V 2630 4650 50  0001 C CNN
-F 3 "" H 2700 4650 50  0000 C CNN
-	1    2700 4650
-	-1   0    0    1
-$EndComp
-$Comp
-L +BATT #PWR08
-U 1 1 5D63FB11
-P 2700 4450
-F 0 "#PWR08" H 2700 4300 50  0001 C CNN
-F 1 "+BATT" H 2700 4590 50  0000 C CNN
-F 2 "" H 2700 4450 50  0000 C CNN
-F 3 "" H 2700 4450 50  0000 C CNN
-	1    2700 4450
-	1    0    0    -1
-$EndComp
-$Comp
-L C C2
-U 1 1 5D236E96
-P 3850 3500
-F 0 "C2" H 3875 3600 50  0000 L CNN
-F 1 "1uF" H 3875 3400 50  0000 L CNN
-F 2 "Capacitors_SMD:C_0805_HandSoldering" H 3888 3350 50  0001 C CNN
-F 3 "" H 3850 3500 50  0000 C CNN
-	1    3850 3500
-	1    0    0    -1
-$EndComp
-Text Label 4900 4200 0    60   ~ 0
-RST
-Text Label 6150 3800 2    60   ~ 0
-TCK
-Text Label 6150 4000 2    60   ~ 0
-TDI
-$Comp
-L GND #PWR09
-U 1 1 5DD8F695
-P 6150 3900
-F 0 "#PWR09" H 6150 3650 50  0001 C CNN
-F 1 "GND" H 6150 3750 50  0000 C CNN
-F 2 "" H 6150 3900 50  0000 C CNN
-F 3 "" H 6150 3900 50  0000 C CNN
-	1    6150 3900
-	0    -1   -1   0
-$EndComp
-$Comp
-L +BATT #PWR010
-U 1 1 5DD8F89B
-P 6150 4100
-F 0 "#PWR010" H 6150 3950 50  0001 C CNN
-F 1 "+BATT" H 6150 4240 50  0000 C CNN
-F 2 "" H 6150 4100 50  0000 C CNN
-F 3 "" H 6150 4100 50  0000 C CNN
-	1    6150 4100
-	0    1    1    0
-$EndComp
 $Comp
 L D_Schottky D57
@@
 $EndComp
 $Comp
-L SW_SPDT SW1
-U 1 1 5DDE22CA
-P 2350 3250
-F 0 "SW1" H 2350 3420 50  0000 C CNN
-F 1 "SW_SPDT" H 2350 3050 50  0000 C CNN
-F 2 "VineBadge2020:JS202011JAQN-Handsolder" H 2350 3250 50  0001 C CNN
-F 3 "" H 2350 3250 50  0000 C CNN
-	1    2350 3250
-	1    0    0    -1
-$EndComp
-$Comp
 L SW_Push SW2
 U 1 1 5DDE23FD
@@
 F 0 "SW2" H 2950 4950 50  0000 L CNN
 F 1 "SW_Push" H 2900 4790 50  0000 C CNN
-F 2 "VineBadge2020:SW_SPST_EVQPE1_Handsolder" H 2900 5050 50  0001 C CNN
+F 2 "Buttons_Switches_SMD:SW_SPST_TL3342" H 2900 5050 50  0001 C CNN
 F 3 "" H 2900 5050 50  0000 C CNN
 	1    2900 4850
@@
 Wire Wire Line
 	16250 3800 16250 4200
-Wire Wire Line
-	2550 3150 2850 3150
-Wire Wire Line
-	3350 3350 3150 3350
-Wire Wire Line
-	3650 3350 4050 3350
-Connection ~ 4900 4200
-Connection ~ 6150 4000
-Connection ~ 6150 3800
-Wire Wire Line
-	5350 4200 4900 4200
-Wire Wire Line
-	5750 4100 6150 4100
-Wire Wire Line
-	5750 4000 6150 4000
-Wire Wire Line
-	5750 3900 6150 3900
-Wire Wire Line
-	5750 3800 6150 3800
-Wire Wire Line
-	2850 3150 2850 3350
-Wire Wire Line
-	1650 3250 1650 3350
-Wire Wire Line
-	2150 3250 1650 3250
-Wire Wire Line
-	2700 4850 2700 4800
-Wire Wire Line
-	2700 4450 2700 4500
 Connection ~ 2400 4850
 Connection ~ 4700 2600
@@
 	7000 3050 12350 3050
 Wire Wire Line
-	2050 1850 2050 1900
-Connection ~ 2050 1500
-Wire Wire Line
 	4700 3050 4700 3100
 Connection ~ 4700 2700
 Wire Wire Line
 	4700 2750 4700 2700
-Connection ~ 3850 3650
-Connection ~ 3850 3350
-Wire Wire Line
-	4050 3650 4050 3700
-Wire Wire Line
-	1650 3650 4050 3650
 Connection ~ 7550 4200
 Connection ~ 16250 1500
@@
 	2050 1500 2150 1500
 Wire Wire Line
-	2050 1400 2050 1550
+	2050 1500 2050 1400
+Wire Wire Line
+	3850 3900 3850 3850
+Wire Wire Line
+	3850 3850 3650 3850
+Wire Wire Line
+	3350 3850 3050 3850
+Wire Wire Line
+	3050 3850 3050 3750
+Wire Wire Line
+	3350 3350 3050 3350
+Wire Wire Line
+	3050 3350 3050 3450
+Wire Wire Line
+	3650 3350 3850 3350
 $EndSCHEMATC

Commit message: kfdjkd
Parts:
- removed F1: Fuse, Fuse_Holders_and_Fuses:Fuse_SMD1206_Reflow, symbol Fuse
- added F1: Polyfuse, Resistors_SMD:R_0603_HandSoldering, symbol Polyfuse
Connections:
- net GND: now also F1.1
- net at BT1.2 (-): now also F1.2
Changed lines of the file:
@@
 $EndComp
 $Comp
-L GND #PWR01
+L GND #PWR2
 U 1 1 5D1D409B
 P 2050 2750
-F 0 "#PWR01" H 2050 2500 50  0001 C CNN
+F 0 "#PWR2" H 2050 2500 50  0001 C CNN
 F 1 "GND" H 2050 2600 50  0000 C CNN
 F 2 "" H 2050 2750 50  0000 C CNN
@@
 $EndComp
 $Comp
-L +BATT #PWR02
+L +BATT #PWR1
 U 1 1 5D1D40B1
 P 2050 1400
-F 0 "#PWR02" H 2050 1250 50  0001 C CNN
+F 0 "#PWR1" H 2050 1250 50  0001 C CNN
 F 1 "+BATT" H 2050 1540 50  0000 C CNN
 F 2 "" H 2050 1400 50  0000 C CNN
@@
 $EndComp
 $Comp
-L GND #PWR03
+L GND #PWR5
 U 1 1 5D236972
 P 3850 3900
-F 0 "#PWR03" H 3850 3650 50  0001 C CNN
+F 0 "#PWR5" H 3850 3650 50  0001 C CNN
 F 1 "GND" H 3850 3750 50  0000 C CNN
 F 2 "" H 3850 3900 50  0000 C CNN
@@
 $EndComp
 $Comp
-L +BATT #PWR04
+L +BATT #PWR4
 U 1 1 5D236A0E
 P 3850 3350
-F 0 "#PWR04" H 3850 3200 50  0001 C CNN
+F 0 "#PWR4" H 3850 3200 50  0001 C CNN
 F 1 "+BATT" H 3850 3490 50  0000 C CNN
 F 2 "" H 3850 3350 50  0000 C CNN
@@
 	1    3850 3350
 	1    0    0    -1
-$EndComp
-$Comp
-L Fuse F1
-U 1 1 5D237CDD
-P 3500 3850
-F 0 "F1" V 3600 3850 50  0000 C CNN
-F 1 "Fuse" V 3425 3850 50  0000 C CNN
-F 2 "Fuse_Holders_and_Fuses:Fuse_SMD1206_Reflow" V 3430 3850 50  0001 C CNN
-F 3 "" H 3500 3850 50  0000 C CNN
-	1    3500 3850
-	0    1    1    0
 $EndComp
 $Comp
@@
 0.3
 $Comp
-L +BATT #PWR05
+L +BATT #PWR3
 U 1 1 5D1D5CCC
 P 4700 3100
-F 0 "#PWR05" H 4700 2950 50  0001 C CNN
+F 0 "#PWR3" H 4700 2950 50  0001 C CNN
 F 1 "+BATT" H 4700 3240 50  0000 C CNN
 F 2 "" H 4700 3100 50  0000 C CNN
@@
 $EndComp
 $Comp
-L GND #PWR06
+L GND #PWR6
 U 1 1 5D63930F
 P 3400 5050
-F 0 "#PWR06" H 3400 4800 50  0001 C CNN
+F 0 "#PWR6" H 3400 4800 50  0001 C CNN
 F 1 "GND" H 3400 4900 50  0000 C CNN
 F 2 "" H 3400 5050 50  0000 C CNN
@@
 	2050 1500 2050 1400
 Wire Wire Line
-	3850 3900 3850 3850
-Wire Wire Line
-	3850 3850 3650 3850
-Wire Wire Line
-	3350 3850 3050 3850
+	3850 3850 3850 3900
 Wire Wire Line
 	3050 3850 3050 3750
@@
 Wire Wire Line
 	3650 3350 3850 3350
+$Comp
+L Polyfuse F1
+U 1 1 5E409A2D
+P 3450 3850
+F 0 "F1" V 3350 3850 50  0000 C CNN
+F 1 "Polyfuse" V 3550 3850 50  0000 C CNN
+F 2 "Resistors_SMD:R_0603_HandSoldering" H 3500 3650 50  0001 L CNN
+F 3 "" H 3450 3850 50  0001 C CNN
+	1    3450 3850
+	0    1    1    0
+$EndComp
+Wire Wire Line
+	3050 3850 3300 3850
+Wire Wire Line
+	3600 3850 3850 3850
 $EndSCHEMATC
